Commit message: updated stairs urdf

File: models/stairs_step_0.02.urdf (robot description, URDF)
Before this commit: robot step, 1 links, 0 joints
Links:
- link step_1: geometry collision box size=0.5 0.5 0.02; visual box size=0.5 0.5 0.02

File: models/stairs_step_0.04.urdf (robot description, URDF)
Before this commit: robot step, 1 links, 0 joints
Links:
- link step_1: geometry collision box size=0.5 0.5 0.04; visual box size=0.5 0.5 0.04
